File: cthruv2.kicad_sch (KiCad schematic)
At the start: 9 parts, among them J1 USB_C_Receptacle, J2 Conn_01x03, J3 Conn_01x05, J7 VBUS, J8 Conn_01x05, P1 USB_C_Plug

Commit message: v3: rerouted pin header pinout, improved routing
Parts:
- J1: LCSC_ID (none) -> C709359
- P1: LCSC_ID (none) -> C319150
- R1: LCSC_ID (none) -> C175856
- R2: LCSC_ID (none) -> C25803
- R3: LCSC_ID (none) -> C25804
Connections:
- net CC2: now also J3.4 (Pin_4), J3.5 (Pin_5); no longer J8.1 (Pin_1), J8.2 (Pin_2)
- net GND: now also J1.S1 (SHIELD), P1.S1 (SHIELD)
- net SBU2: now also J8.1 (Pin_1), J8.2 (Pin_2); no longer J3.4 (Pin_4), J3.5 (Pin_5)
